File: cape/cape_rev_a.brd (EAGLE design)
At the start: 100 x 80 mm, 35 parts, among them IC1 MAX3042BEUE, IC10 MAX3042BEUE, IC11 MAX3042BEUE, IC12 MAX3042BEUE, IC13 MAX3042BEUE, IC14 MAX3042BEUE, IC15 MAX3042BEUE, IC16 MAX3042BEUE, IC2 MAX3042BEUE, IC3 MAX3042BEUE, IC4 MAX3042BEUE, IC5 MAX3042BEUE, IC6 MAX3042BEUE, IC7 MAX3042BEUE, IC8 MAX3042BEUE, IC9 MAX3042BEUE

Commit message: Made some progress on layout for cape
Parts:
- removed U$1: BEAGLEBONE_OUTLINEDOCU_OUTLINE, microbuilder:BEAGLEBONE_OUTLINE_DOCU
- added U$3: BEAGLEBONE_OUTLINEDOCU_OUTLINE, microbuilder:BEAGLEBONE_OUTLINE_DOCU
- moved C16 317.4 mm to (74.0, 112.9), turned to 180 degrees
- moved C15 307.8 mm to (74.0, 106.0), turned to 180 degrees
- moved C14 298.0 mm to (74.0, 98.9), turned to 180 degrees
- moved C13 288.4 mm to (74.0, 92.0), turned to 180 degrees
- moved C12 278.7 mm to (74.0, 84.9), turned to 180 degrees
- moved C11 269.1 mm to (74.0, 78.0), turned to 180 degrees
- moved C10 259.4 mm to (74.0, 71.0), turned to 180 degrees
- moved C9 250.0 mm to (74.0, 64.1), turned to 180 degrees
- moved IC16 246.7 mm to (79.1, 115.5), turned to 90 degrees
- moved C8 240.4 mm to (74.0, 57.0), turned to 180 degrees
- moved IC15 232.9 mm to (79.1, 108.6), turned to 90 degrees
- moved C7 231.0 mm to (74.0, 50.1), turned to 180 degrees
- moved C6 221.4 mm to (74.0, 43.0), turned to 180 degrees
- moved IC14 219.0 mm to (79.1, 101.5), turned to 90 degrees
- moved C5 212.1 mm to (74.0, 36.2), turned to 180 degrees
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Connections:
- net 10A+: now also U$2.P10-1
- net 10A-: now also U$2.P10-2
- net 10B+: now also U$2.P10-3
- net 10B-: now also U$2.P10-6
- net 10C+: now also U$2.P10-4
- net 10C-: now also U$2.P10-5
- net 10D+: now also U$2.P10-7
- net 10D-: now also U$2.P10-8
- net 11A+: now also U$2.P11-1
- net 11A-: now also U$2.P11-2
- net 11B+: now also U$2.P11-3
- net 11B-: now also U$2.P11-6
- net 11C+: now also U$2.P11-4
- net 11C-: now also U$2.P11-5
- net 11D+: now also U$2.P11-7
- net 11D-: now also U$2.P11-8
- net 12A+: now also U$2.P12-1
- net 12A-: now also U$2.P12-2
- net 12B+: now also U$2.P12-3
- net 12B-: now also U$2.P12-6
- net 12C+: now also U$2.P12-4
- net 12C-: now also U$2.P12-5
- net 12D+: now also U$2.P12-7
- net 12D-: now also U$2.P12-8
- net 13A+: now also U$2.P13-1
- net 13A-: now also U$2.P13-2
- net 13B+: now also U$2.P13-3
- net 13B-: now also U$2.P13-6
- net 13C+: now also U$2.P13-4
- net 13C-: now also U$2.P13-5
- net 13D+: now also U$2.P13-7
- net 13D-: now also U$2.P13-8
- net 14A+: now also U$2.P14-1
- net 14A-: now also U$2.P14-2
- net 14B+: now also U$2.P14-3
- net 14B-: now also U$2.P14-6
- net 14C+: now also U$2.P14-4
- net 14C-: now also U$2.P14-5
- net 14D+: now also U$2.P14-7
- net 14D-: now also U$2.P14-8
- net 15A+: now also U$2.P15-1
- net 15A-: now also U$2.P15-2
- net 15B+: now also U$2.P15-3
- net 15B-: now also U$2.P15-6
- net 15C+: now also U$2.P15-4
- net 15C-: now also U$2.P15-5
- net 15D+: now also U$2.P15-7
- net 15D-: now also U$2.P15-8
- net 16A+: now also U$2.P16-1
- net 16A-: now also U$2.P16-2
- net 16B+: now also U$2.P16-3
- net 16B-: now also U$2.P16-6
- net 16C+: now also U$2.P16-4
- net 16C-: now also U$2.P16-5
- net 16D+: now also U$2.P16-7
- net 16D-: now also U$2.P16-8
- net 2A+: now also U$2.P2-1
- net 2A-: now also U$2.P2-2
- net 2B+: now also U$2.P2-3
- net 2B-: now also U$2.P2-6
- net 2C+: now also U$2.P2-4
- net 2C-: now also U$2.P2-5
- net 2D+: now also U$2.P2-7
- net 2D-: now also U$2.P2-8
- net 3A+: now also U$2.P3-1
- net 3A-: now also U$2.P3-2
- net 3B+: now also U$2.P3-3
- net 3B-: now also U$2.P3-6
- net 3C+: now also U$2.P3-4
- net 3C-: now also U$2.P3-5
- net 3D+: now also U$2.P3-7
- net 3D-: now also U$2.P3-8
- net 4A+: now also U$2.P4-1
- net 4A-: now also U$2.P4-2
- net 4B+: now also U$2.P4-3
- net 4B-: now also U$2.P4-6
- net 4C+: now also U$2.P4-4
- net 4C-: now also U$2.P4-5
- net 4D+: now also U$2.P4-7
- net 4D-: now also U$2.P4-8
- net 5A+: now also U$2.P5-1
- net 5A-: now also U$2.P5-2
- net 5B+: now also U$2.P5-3
- net 5B-: now also U$2.P5-6
- net 5C+: now also U$2.P5-4
- net 5C-: now also U$2.P5-5
- net 5D+: now also U$2.P5-7
- net 5D-: now also U$2.P5-8
- net 6A+: now also U$2.P6-1
- net 6A-: now also U$2.P6-2
- net 6B+: now also U$2.P6-3
- net 6B-: now also U$2.P6-6
- net 6C+: now also U$2.P6-4
- net 6C-: now also U$2.P6-5
- net 6D+: now also U$2.P6-7
- net 6D-: now also U$2.P6-8
- net 7A+: now also U$2.P7-1
- net 7A-: now also U$2.P7-2
- net 7B+: now also U$2.P7-3
- net 7B-: now also U$2.P7-6
- net 7C+: now also U$2.P7-4
- net 7C-: now also U$2.P7-5
- net 7D+: now also U$2.P7-7
- net 7D-: now also U$2.P7-8
- net 8A+: now also U$2.P8-1
- net 8A-: now also U$2.P8-2
- net 8B+: now also U$2.P8-3
- net 8B-: now also U$2.P8-6
- net 8C+: now also U$2.P8-4
- net 8C-: now also U$2.P8-5
- net 8D+: now also U$2.P8-7
- net 8D-: now also U$2.P8-8
- net 9A+: now also U$2.P9-1
- net 9A-: now also U$2.P9-2
- net 9B+: now also U$2.P9-3
- net 9B-: now also U$2.P9-6
- net 9C+: now also U$2.P9-4
- net 9C-: now also U$2.P9-5
- net 9D+: now also U$2.P9-7
- net 9D-: now also U$2.P9-8
- net GND: now also U$3.1, U$3.2, U$3.47, U$3.48, U$3.89, U$3.90, U$3.91, U$3.92; no longer U$1.1, U$1.2, U$1.47, U$1.48, U$1.89, U$1.90, U$1.91, U$1.92
- net GNDA_ADC: now also U$3.80; no longer U$1.80
- net N$1: now also IC10.1, IC11.1, IC12.1, IC13.1, IC14.1, IC15.1, IC16.1, IC2.1, IC3.1, IC4.1, IC5.1, IC6.1, IC7.1, IC8.1, IC9.1
- net N$2: now also IC10.7, IC11.7, IC12.7, IC13.7, IC14.7, IC15.7, IC16.7, IC2.7, IC3.7, IC4.7, IC5.7, IC6.7, IC7.7, IC8.7, IC9.7
- net N$3: now also IC10.9, IC11.9, IC12.9, IC13.9, IC14.9, IC15.9, IC16.9, IC2.9, IC3.9, IC4.9, IC5.9, IC6.9, IC7.9, IC8.9, IC9.9
- net N$4: now also IC10.15, IC11.15, IC12.15, IC13.15, IC14.15, IC15.15, IC16.15, IC2.15, IC3.15, IC4.15, IC5.15, IC6.15, IC7.15, IC8.15, IC9.15
- net SYS_5V: now also U$3.53, U$3.54; no longer U$1.53, U$1.54
- net VCC: now also IC10.12, IC10.4, IC11.12, IC11.4, IC12.12, IC12.4, IC13.12, IC13.4, IC14.12, IC14.4, IC15.12, IC15.4, IC16.12, IC16.4, IC2.12, IC2.4, IC3.12, IC3.4, IC4.12, IC4.4, IC5.12, IC5.4, IC6.12, IC6.4, IC7.12, IC7.4, IC8.12, IC8.4, IC9.12, IC9.4
- net VDD_3V3EXP: now also U$3.49, U$3.50; no longer U$1.49, U$1.50
- net VDD_5V: now also U$3.51, U$3.52; no longer U$1.51, U$1.52
- net VDD_ADC: now also U$3.78; no longer U$1.78
Routing:
- net VCC: track 0.00 -> 90.0 mm
- net 1D-: track 0.00 -> 43.6 mm, vias 0 -> 1
- net 1D+: track 0.00 -> 42.0 mm, vias 0 -> 1
- net 5D-: track 0.00 -> 39.9 mm, vias 0 -> 1
- net 11D-: track 0.00 -> 39.9 mm, vias 0 -> 1
- net 9D-: track 0.00 -> 39.9 mm, vias 0 -> 1
- net 15D-: track 0.00 -> 39.9 mm, vias 0 -> 1
- net 13D-: track 0.00 -> 39.9 mm, vias 0 -> 1
- net 3D-: track 0.00 -> 39.9 mm, vias 0 -> 1
- net 3D+: track 0.00 -> 38.6 mm, vias 0 -> 1
- net 5D+: track 0.00 -> 38.6 mm, vias 0 -> 1
- net 15D+: track 0.00 -> 38.5 mm, vias 0 -> 1
- net 9D+: track 0.00 -> 38.5 mm, vias 0 -> 1
- net 13D+: track 0.00 -> 38.5 mm, vias 0 -> 1
- net 11D+: track 0.00 -> 38.5 mm, vias 0 -> 1
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Other:
- board size 100 x 80 mm -> 116.4 x 127.2 mm

Commit message: More routing
Routing:
- net VCC: track 90.0 -> 201.3 mm
- net VCC3: track 21.8 -> 0.00 mm
- net VCC2: track 21.8 -> 0.00 mm
- net VCC1: track 21.8 -> 0.00 mm
- net VCC5: track 21.8 -> 0.00 mm
- net 8D-: track 19.2 -> 21.6 mm, vias 0 -> 1
- net 8C+: track 18.0 -> 20.4 mm, vias 0 -> 1
- net 8C-: track 15.6 -> 17.9 mm, vias 0 -> 1
- net 7D-: track 37.7 -> 39.9 mm, vias 0 -> 1
- net 7C-: track 28.5 -> 30.6 mm, vias 0 -> 1
- net 7D+: track 36.4 -> 38.6 mm, vias 0 -> 1
- net 7C+: track 25.0 -> 27.1 mm, vias 0 -> 1
- net 8D+: track 16.3 -> 18.1 mm, vias 0 -> 1
- net 9D-: track 39.9 -> 40.6 mm
