File: cape/cape_rev_a.sch (EAGLE design)
At the start: 35 parts, among them IC1 MAX3042BEUE, IC10 MAX3042BEUE, IC11 MAX3042BEUE, IC12 MAX3042BEUE, IC13 MAX3042BEUE, IC14 MAX3042BEUE, IC15 MAX3042BEUE, IC16 MAX3042BEUE, IC2 MAX3042BEUE, IC3 MAX3042BEUE, IC4 MAX3042BEUE, IC5 MAX3042BEUE, IC6 MAX3042BEUE, IC7 MAX3042BEUE, IC8 MAX3042BEUE, IC9 MAX3042BEUE

Commit message: Made some progress on layout for cape
Parts:
- removed U$1: BEAGLEBONE_OUTLINEDOCU_OUTLINE, microbuilder:BEAGLEBONE_OUTLINEDOCU_OUTLINE
- added U$3: BEAGLEBONE_OUTLINEDOCU_OUTLINE, microbuilder:BEAGLEBONE_OUTLINEDOCU_OUTLINE
Connections:
- net 10A+: now also U$2.10-1
- net 10A-: now also U$2.10-2
- net 10B+: now also U$2.10-3
- net 10B-: now also U$2.10-6
- net 10C+: now also U$2.10-4
- net 10C-: now also U$2.10-5
- net 10D+: now also U$2.10-7
- net 10D-: now also U$2.10-8
- net 11A+: now also U$2.11-1
- net 11A-: now also U$2.11-2
- net 11B+: now also U$2.11-3
- net 11B-: now also U$2.11-6
- net 11C+: now also U$2.11-4
- net 11C-: now also U$2.11-5
- net 11D+: now also U$2.11-7
- net 11D-: now also U$2.11-8
- net 12A+: now also U$2.12-1
- net 12A-: now also U$2.12-2
- net 12B+: now also U$2.12-3
- net 12B-: now also U$2.12-6
- net 12C+: now also U$2.12-4
- net 12C-: now also U$2.12-5
- net 12D+: now also U$2.12-7
- net 12D-: now also U$2.12-8
- net 13A+: now also U$2.13-1
- net 13A-: now also U$2.13-2
- net 13B+: now also U$2.13-3
- net 13B-: now also U$2.13-6
- net 13C+: now also U$2.13-4
- net 13C-: now also U$2.13-5
- net 13D+: now also U$2.13-7
- net 13D-: now also U$2.13-8
- net 14A+: now also U$2.14-1
- net 14A-: now also U$2.14-2
- net 14B+: now also U$2.14-3
- net 14B-: now also U$2.14-6
- net 14C+: now also U$2.14-4
- net 14C-: now also U$2.14-5
- net 14D+: now also U$2.14-7
- net 14D-: now also U$2.14-8
- net 15A+: now also U$2.15-1
- net 15A-: now also U$2.15-2
- net 15B+: now also U$2.15-3
- net 15B-: now also U$2.15-6
- net 15C+: now also U$2.15-4
- net 15C-: now also U$2.15-5
- net 15D+: now also U$2.15-7
- net 15D-: now also U$2.15-8
- net 16A+: now also U$2.16-1
- net 16A-: now also U$2.16-2
- net 16B+: now also U$2.16-3
- net 16B-: now also U$2.16-6
- net 16C+: now also U$2.16-4
- net 16C-: now also U$2.16-5
- net 16D+: now also U$2.16-7
- net 16D-: now also U$2.16-8
- net 2A+: now also U$2.2-1
- net 2A-: now also U$2.2-2
- net 2B+: now also U$2.2-3
- net 2B-: now also U$2.2-6
- net 2C+: now also U$2.2-4
- net 2C-: now also U$2.2-5
- net 2D+: now also U$2.2-7
- net 2D-: now also U$2.2-8
- net 3A+: now also U$2.3-1
- net 3A-: now also U$2.3-2
- net 3B+: now also U$2.3-3
- net 3B-: now also U$2.3-6
- net 3C+: now also U$2.3-4
- net 3C-: now also U$2.3-5
- net 3D+: now also U$2.3-7
- net 3D-: now also U$2.3-8
- net 4A+: now also U$2.4-1
- net 4A-: now also U$2.4-2
- net 4B+: now also U$2.4-3
- net 4B-: now also U$2.4-6
- net 4C+: now also U$2.4-4
- net 4C-: now also U$2.4-5
- net 4D+: now also U$2.4-7
- net 4D-: now also U$2.4-8
- net 5A+: now also U$2.5-1
- net 5A-: now also U$2.5-2
- net 5B+: now also U$2.5-3
- net 5B-: now also U$2.5-6
- net 5C+: now also U$2.5-4
- net 5C-: now also U$2.5-5
- net 5D+: now also U$2.5-7
- net 5D-: now also U$2.5-8
- net 6A+: now also U$2.6-1
- net 6A-: now also U$2.6-2
- net 6B+: now also U$2.6-3
- net 6B-: now also U$2.6-6
- net 6C+: now also U$2.6-4
- net 6C-: now also U$2.6-5
- net 6D+: now also U$2.6-7
- net 6D-: now also U$2.6-8
- net 7A+: now also U$2.7-1
- net 7A-: now also U$2.7-2
- net 7B+: now also U$2.7-3
- net 7B-: now also U$2.7-6
- net 7C+: now also U$2.7-4
- net 7C-: now also U$2.7-5
- net 7D+: now also U$2.7-7
- net 7D-: now also U$2.7-8
- net 8A+: now also U$2.8-1
- net 8A-: now also U$2.8-2
- net 8B+: now also U$2.8-3
- net 8B-: now also U$2.8-6
- net 8C+: now also U$2.8-4
- net 8C-: now also U$2.8-5
- net 8D+: now also U$2.8-7
- net 8D-: now also U$2.8-8
- net 9A+: now also U$2.9-1
- net 9A-: now also U$2.9-2
- net 9B+: now also U$2.9-3
- net 9B-: now also U$2.9-6
- net 9C+: now also U$2.9-4
- net 9C-: now also U$2.9-5
- net 9D+: now also U$2.9-7
- net 9D-: now also U$2.9-8
- net GND: now also IC10.GND, IC11.GND, IC12.GND, IC13.GND, IC14.GND, IC15.GND, IC16.GND, IC2.GND, IC3.GND, IC4.GND, IC5.GND, IC6.GND, IC7.GND, IC8.GND, IC9.GND
- net N$1: now also IC10.T1IN, IC11.T1IN, IC12.T1IN, IC13.T1IN, IC14.T1IN, IC15.T1IN, IC16.T1IN, IC2.T1IN, IC3.T1IN, IC4.T1IN, IC5.T1IN, IC6.T1IN, IC7.T1IN, IC8.T1IN, IC9.T1IN
- net N$2: now also IC10.T2IN, IC11.T2IN, IC12.T2IN, IC13.T2IN, IC14.T2IN, IC15.T2IN, IC16.T2IN, IC2.T2IN, IC3.T2IN, IC4.T2IN, IC5.T2IN, IC6.T2IN, IC7.T2IN, IC8.T2IN, IC9.T2IN
- net N$3: now also IC10.T3IN, IC11.T3IN, IC12.T3IN, IC13.T3IN, IC14.T3IN, IC15.T3IN, IC16.T3IN, IC2.T3IN, IC3.T3IN, IC4.T3IN, IC5.T3IN, IC6.T3IN, IC7.T3IN, IC8.T3IN, IC9.T3IN
- net N$4: now also IC10.T4IN, IC11.T4IN, IC12.T4IN, IC13.T4IN, IC14.T4IN, IC15.T4IN, IC16.T4IN, IC2.T4IN, IC3.T4IN, IC4.T4IN, IC5.T4IN, IC6.T4IN, IC7.T4IN, IC8.T4IN, IC9.T4IN
- net VCC: now also IC10.EN12, IC10.EN34, IC10.VCC, IC11.EN12, IC11.EN34, IC11.VCC, IC12.EN12, IC12.EN34, IC12.VCC, IC13.EN12, IC13.EN34, IC13.VCC, IC14.EN12, IC14.EN34, IC14.VCC, IC15.EN12, IC15.EN34, IC15.VCC, IC16.EN12, IC16.EN34, IC16.VCC, IC2.EN12, IC2.EN34, IC2.VCC, IC3.EN12, IC3.EN34, IC3.VCC, IC4.EN12, IC4.EN34, IC4.VCC, IC5.EN12, IC5.EN34, IC5.VCC, IC6.EN12, IC6.EN34, IC6.VCC, IC7.EN12, IC7.EN34, IC7.VCC, IC8.EN12, IC8.EN34, IC8.VCC, IC9.EN12, IC9.EN34, IC9.VCC
Other:
- moved on the sheet: IC14

Commit message: Mostly done with the receiver
Connections:
- new net CLOCK0: U$3.GPIO2_22
- new net CLOCK1: U$3.GPIO1_13
Changed lines of the file:
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@@
+</segment>
+</net>
+<net name="CLOCK1" class="0">
+<segment>
+<pinref part="U$3" gate="G$1" pin="GPIO1_13"/>
+<wire x1="2.54" y1="127" x2="-7.62" y2="127" width="0.1524" layer="91"/>
+<label x="-12.7" y="127" size="1.778" layer="95"/>
+</segment>
+</net>
+<net name="CLOCK0" class="0">
+<segment>
+<pinref part="U$3" gate="G$1" pin="GPIO2_22"/>
+<wire x1="2.54" y1="106.68" x2="-7.62" y2="106.68" width="0.1524" layer="91"/>
+<label x="-12.7" y="106.68" size="1.778" layer="95"/>
 </segment>
 </net>

Commit message: Almost done with cape routing
Parts:
- added C17: 0.1uF, SparkFun-Passives:CAP0603-CAP
- added U17: SN74LV245, microbuilder:74LCX245
- renumbered IC1 to U1, IC10 to U10, IC11 to U11, IC12 to U12, IC13 to U13, IC14 to U14, IC15 to U15, IC16 to U16, IC2 to U2, IC3 to U3, IC4 to U4, IC5 to U5, IC6 to U6, IC7 to U7, IC8 to U8, IC9 to U9
Connections:
- removed net CLOCK0: U$3.GPIO2_22
- removed net CLOCK1: U$3.GPIO1_13
- removed net N$1: U1.T1IN, U10.T1IN, U11.T1IN, U12.T1IN, U13.T1IN, U14.T1IN, U15.T1IN, U16.T1IN, U2.T1IN, U3.T1IN, U4.T1IN, U5.T1IN, U6.T1IN, U7.T1IN, U8.T1IN, U9.T1IN
- removed net N$2: U1.T2IN, U10.T2IN, U11.T2IN, U12.T2IN, U13.T2IN, U14.T2IN, U15.T2IN, U16.T2IN, U2.T2IN, U3.T2IN, U4.T2IN, U5.T2IN, U6.T2IN, U7.T2IN, U8.T2IN, U9.T2IN
- removed net N$3: U1.T3IN, U10.T3IN, U11.T3IN, U12.T3IN, U13.T3IN, U14.T3IN, U15.T3IN, U16.T3IN, U2.T3IN, U3.T3IN, U4.T3IN, U5.T3IN, U6.T3IN, U7.T3IN, U8.T3IN, U9.T3IN
- removed net N$4: U1.T4IN, U10.T4IN, U11.T4IN, U12.T4IN, U13.T4IN, U14.T4IN, U15.T4IN, U16.T4IN, U2.T4IN, U3.T4IN, U4.T4IN, U5.T4IN, U6.T4IN, U7.T4IN, U8.T4IN, U9.T4IN
- new net CK0-1: U1.T4IN, U17.B1, U2.T4IN
- new net CK0-2: U17.B2, U3.T4IN, U4.T4IN
- new net CK0-3: U17.B3, U5.T4IN, U6.T4IN
- new net CK0-4: U17.B4, U7.T4IN, U8.T4IN
- new net CK1-1: U10.T4IN, U17.B5, U9.T4IN
- new net CK1-2: U11.T4IN, U12.T4IN, U17.B6
- new net CK1-3: U13.T4IN, U14.T4IN, U17.B7
- new net CK1-4: U15.T4IN, U16.T4IN, U17.B8
- new net PRU0: U$3.GPIO1_13, U17.A1, U17.A2, U17.A3, U17.A4
- new net PRU1: U$3.GPIO2_22, U17.A5, U17.A6, U17.A7, U17.A8
- new net S0: U$3.TIMER7, U1.T1IN
- new net S1: U$3.GPIO1_12, U1.T2IN
- new net S10: U$3.UART3_CTSN, U4.T2IN
- new net S11: U$3.UART3_RTSN, U4.T3IN
- new net S12: U$3.UART5_RXD, U5.T1IN
- new net S13: U$3.GPIO2_11, U5.T2IN
- new net S14: U$3.GPIO2_13, U5.T3IN
- new net S15: U$3.GPIO2_7, U6.T1IN
- new net S16: U$3.GPIO2_9, U6.T2IN
- new net S17: U$3.GPIO2_6, U6.T3IN
- new net S18: U$3.GPIO2_8, U7.T1IN
- new net S19: U$3.GPIO2_12, U7.T2IN
- new net S2: U$3.TIMER6, U1.T3IN
- new net S20: U$3.GPIO2_10, U7.T3IN
- new net S21: U$3.UART5_TXD, U8.T1IN
- new net S22: U$3.UART4_RTSN, U8.T2IN
- new net S23: U$3.UART4_CTSN, U8.T3IN
- new net S24: U$3.UART5_CTSN, U9.T1IN
- new net S25: U$3.EHRPWM2A, U9.T2IN
- new net S26: U$3.GPIO2_23, U9.T3IN
- new net S27: U$3.GPIO0_27, U10.T1IN
- new net S28: U$3.EHRPWM2B, U10.T2IN
- new net S29: U$3.GPIO1_15, U10.T3IN
- new net S3: U$3.GPIO0_26, U2.T1IN
- new net S30: U$3.TIMER5, U11.T1IN
- new net S31: U$3.GPIO0_7, U11.T2IN
- new net S32: U$3.TIMER4, U11.T3IN
- new net S33: U$3.CLKOUT2, U12.T1IN
- new net S34: U$3.SPI1_DI, U12.T2IN
- new net S35: U$3.SPI1_SCLK, U12.T3IN
- new net S36: U$3.SPI1_DO, U13.T1IN
- new net S37: U$3.SPI1_CS0, U13.T2IN
- new net S38: U$3.GPIO3_19, U13.T3IN
- new net S39: U$3.GPIO3_21, U14.T1IN
- new net S4: U$3.GPIO2_1, U2.T2IN
- new net S40: U$3.UART1_TXD, U14.T2IN
- new net S41: U$3.GPIO1_17, U14.T3IN
- new net S42: U$3.EHRPWM1B, U15.T1IN
- new net S43: U$3.EHRPWM1A, U15.T2IN
- new net S44: U$3.GPIO1_16, U15.T3IN
- new net S45: U$3.UART4_TXD, U16.T1IN
- new net S46: U$3.GPIO1_28, U16.T2IN
- new net S47: U$3.UART4_RXD, U16.T3IN
- new net S5: U$3.GPIO1_14, U2.T3IN
- new net S6: U$3.GPIO1_29, U3.T1IN
- new net S7: U$3.GPIO2_25, U3.T2IN
- new net S8: U$3.GPIO2_24, U3.T3IN
- new net S9: U$3.UART5_RTSN, U4.T1IN
- net GND: now also C17.2, U$3.GND@1, U$3.GND@2, U$3.GND@3, U$3.GND@4, U$3.GND@5, U$3.GND@6, U$3.GND@7, U$3.GND@8, U17./OE, U17.GND
- net VCC: now also C17.1, U$3.VDD_5V@1, U$3.VDD_5V@2, U17.T/R, U17.VCC
